Commit message: Moving things into their measured positions

File: src/hros5_description/urdf/modules/head.xacro (robot description, xacro)
@@ -86,5 +86,5 @@
 	<parent link="UpperHeadBase" />
 	<child link="realsense_frame" />
-	<origin xyz="0.0 0.0 0.0" rpy="${pi/2} ${pi} ${pi/2}" />
+	<origin xyz="0.05 -0.05 0.05" rpy="${pi/2} ${pi} ${pi/2}" />
 </joint>
 <link name="realsense_frame" />

File: src/hros5_description/urdf/modules/torso.xacro (robot description, xacro)
@@ -20,5 +20,5 @@
     <parent link="base_link"/>
     <child link="torso"/>
-    <origin xyz="0.0 0.0 0.0" rpy="0.0 0.0 0.0"/>
+    <origin xyz="0.0 0.0 0.033" rpy="0.0 0.0 0.0"/>
 </joint>
 <!--

Commit message: A little cleanup of PrimeSense and R200 sensor configurations

File: src/hros5_description/urdf/modules/head.xacro (robot description, xacro)
@@ -63,9 +63,9 @@
 <!-- Camera properties -->
 <xacro:property name="pi" value="3.1415926535897931" />
-<!-- openni2
+<!-- openni2 / primesense on top of servo -->
 <joint name="camera_rgb_joint" type="fixed">
 	<parent link="UpperHeadBase" />
 	<child link="camera_rgb_optical_frame" />
-	<origin xyz="0.0 0.0 0.0" rpy="${pi/2} ${pi} ${pi/2}" />
+	<origin xyz="0.0 0.0 0.08" rpy="${pi/2} ${pi} ${pi/2}" />
 </joint>
 <link name="camera_rgb_optical_frame" />
@@ -73,5 +73,5 @@
 	<parent link="UpperHeadBase" />
 	<child link="camera_depth_optical_frame" />
-	<origin xyz="0.0 0.0 0.0" rpy="${pi/2} ${pi} ${pi/2}" />
+	<origin xyz="0.0 0.0 0.08" rpy="${pi/2} ${pi} ${pi/2}" />
 </joint>
 <link name="camera_depth_optical_frame" />
@@ -79,8 +79,8 @@
 	<parent link="UpperHeadBase" />
 	<child link="camera_depth_frame_link" />
-	<origin xyz="0.0 0.0 0.0" />
+	<origin xyz="0.0 0.0 0.08" />
 </joint>
 <link name="camera_depth_frame_link" />
--->
+<!-- intel r200 on front of servo -->
 <joint name="r200_frame" type="fixed">
 	<parent link="UpperHeadBase" />
@@ -89,12 +89,4 @@
 </joint>
 <link name="realsense_frame" />
-<!--
-<joint name="camera_color_joint" type="fixed">
-	<parent link="UpperHeadBase" />
-	<child link="camera_color_optical_frame" />
-	<origin xyz="0.0 0.0 0.0" rpy="${pi/2} ${pi} ${pi/2}" />
-</joint>
-<link name="camera_color_optical_frame" />
--->
 <!-- ROS REP LINKS -->
 	<joint name="gaze_joint" type="fixed">
