Commit message: Adjusted Torso Z Origin

File: hros5_common/hros5_description/urdf/modules/torso.xacro (robot description, xacro)
@@ -5,5 +5,5 @@
 		<parent link="base_link"/>
 		<child link="torso"/>
-		<origin xyz="0 0 0.024" rpy="0 0 0"/>
+		<origin xyz="0 0 0.24" rpy="0 0 0"/>
 	</joint>
 	<!-- TORSO -->

Commit message: IMU fixes mainly.

File: hros5_common/hros5_description/urdf/modules/torso.xacro (robot description, xacro)
@@ -5,5 +5,4 @@
 		<parent link="base_link"/>
 		<child link="torso"/>
-		<origin xyz="0 0 0.24" rpy="0 0 0"/>
 	</joint>
 	<!-- TORSO -->
@@ -16,9 +15,8 @@
 		</inertial>
 	</link>
-<!-- IMU properties -->
-<!--
-<joint name="imu_joint" type="floating">
-    <parent link="base_link"/>
-    <child link="torso"/>
+<!-- IMU properties
+<joint name="imu_joint" type="fixed">
+    <parent link="torso"/>
+    <child link="imu_link"/>
     <origin xyz="0.0 0.0 0.033" rpy="0.0 0.0 0.0"/>
 </joint>
@@ -35,5 +33,5 @@
 	<gazebo>
         <plugin filename="libhector_gazebo_ros_imu.so" name="gazebo_ros_imu">
-          <bodyName>torso</bodyName>
+          <bodyName>imu_link</bodyName>
           <updateRate>50</updateRate>
           <serviceName>/hros5/imu_service</serviceName>
