Commit message: mid-dev dump

File: hros5_common/hros5_description/urdf/modules/head.xacro (robot description, xacro)
@@ -82,5 +82,12 @@
 </joint>
 <link name="camera_depth_frame_link" />
-<!-- intel r200 on front of servo -->
+<!-- intel F200 on top of primesense -->
+<joint name="f200_frame" type="fixed">
+	<parent link="UpperHeadBase" />
+	<child link="realsense_frame" />
+	<origin xyz="0.04 0.0 0.120" rpy="${pi/2} ${pi} ${pi/2}" />
+</joint>
+<link name="realsense_frame" />
+<!-- intel r200 on front of servo
 <joint name="r200_frame" type="fixed">
 	<parent link="UpperHeadBase" />
@@ -89,4 +96,5 @@
 </joint>
 <link name="realsense_frame" />
+-->
 <!-- ROS REP LINKS -->
 	<joint name="gaze_joint" type="fixed">

File: hros5_common/hros5_description/urdf/modules/legs.xacro (robot description, xacro)
@@ -6,5 +6,5 @@
 			<child link="${side}Hip"/>
 			<origin xyz="0.0175 ${reflect*0.048} -0.063" rpy="0 0 0"/>
-			<axis xyz="0 0 1"/>
+			<axis xyz="0 0 -1"/>
 			<limit lower="-0.523598776" upper="0.523598776" effort="8.4" velocity="4.712388975"/>
 		</joint>
